File: mm_motor_control.kicad_sch (KiCad schematic)
At the start: 0 parts

Commit message: tp2
Parts:
- added C7: 2.2m, symbol Device:C
- added CEN0: 10n, symbol Device:C
- added CEN1: 1n, symbol Device:C
- added Ctoff0: 22n, symbol Device:C
- added R10, R11: 330m, symbol Device:R
- added REN0, REN1, REN2, REN3: 18K, symbol Device:R
- added REN4: 1.8K, symbol Device:R
- added Rtoff0: 1K, symbol Device:R
- added U3: STSPIN240, Package_DFN_QFN:VQFN-16-1EP_3x3mm_P0.5mm_EP1.8x1.8mm, symbol Driver_Motor:STSPIN240
Connections:
- net EN: now also REN0.1
- net FAULT: now also CEN0.1, REN0.2, U3.13 (EN/FLT)
- net OUT_A1: now also U3.3 (OUTA1)
- net OUT_A2: now also U3.5 (OUTA2)
- net OUT_B1: now also U3.10 (OUTB1)
- net OUT_B2: now also U3.8 (OUTB2)
- net PHASE_A: now also U3.1 (PHA)
- net PHASE_B: now also U3.15 (PHB)
- net PWM_A: now also U3.2 (PWMA)
- net PWM_B: now also U3.16 (PWMB)
- net STBY/RESET: now also CEN1.1, REN1.1, U3.14 (STBY/RESET)
- new net: R10.1, U3.9 (SENSEB)
- new net: REN3.2, Rtoff0.2, U3.12 (TOFF)
- new net: REN2.1, REN4.2, U3.11 (REF)
- new net: R11.1, U3.4 (SENSEA)
- new net: Ctoff0.1, Rtoff0.1
- new net +3.3V: REN1.2
- new net +BATT: C7.1, REN2.2, U3.6 (VS)
- new net GND: C7.2, CEN0.2, CEN1.2, Ctoff0.2, R10.2, R11.2, REN3.1, REN4.1, U3.17 (EPAD), U3.7 (GND)

Commit message: salim
Parts:
- removed CEN1: 1n, symbol Device:C
- removed REN1: 18K, symbol Device:R
- C7: value 2.2m -> 2.2u; footprint (none) -> Capacitor_SMD:C_0603_1608Metric
- CEN0: value 10n -> 1n; footprint (none) -> Capacitor_SMD:C_0603_1608Metric
- Ctoff0: footprint (none) -> Capacitor_SMD:C_0603_1608Metric
- R10, R11: footprint (none) -> Resistor_SMD:R_2512_6332Metric
- REN0, REN2: value 18K -> 10K; footprint (none) -> Resistor_SMD:R_0603_1608Metric
- REN3: value 18K -> 47K; footprint (none) -> Resistor_SMD:R_0603_1608Metric
- REN4: value 1.8K -> 10K; footprint (none) -> Resistor_SMD:R_0603_1608Metric
- Rtoff0: footprint (none) -> Resistor_SMD:R_0603_1608Metric
Changed lines of the file:
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@@
 (kicad_sch (version 20230121) (generator eeschema)
   (paper "A4")
-  (junction (at 67.31 130.81) (diameter 0) (color 0 0 0 0)
-  )
   (junction (at 160.02 111.76) (diameter 0) (color 0 0 0 0)
   )
@@
     (stroke (width 0) (type default))
   )
-  (wire (pts (xy 93.98 130.81) (xy 67.31 130.81))
-    (stroke (width 0) (type default))
-  )
-  (wire (pts (xy 67.31 128.27) (xy 67.31 130.81))
-    (stroke (width 0) (type default))
-  )
   (wire (pts (xy 198.12 81.28) (xy 166.37 81.28))
     (stroke (width 0) (type default))
@@
     (stroke (width 0) (type default))
   )
-  (wire (pts (xy 60.96 130.81) (xy 67.31 130.81))
-    (stroke (width 0) (type default))
-  )
   (wire (pts (xy 110.49 77.47) (xy 138.43 77.47))
     (stroke (width 0) (type default))
@@
     (stroke (width 0) (type default))
   )
-  (wire (pts (xy 67.31 140.97) (xy 67.31 144.78))
-    (stroke (width 0) (type default))
-  )
-  (wire (pts (xy 67.31 133.35) (xy 67.31 130.81))
-    (stroke (width 0) (type default))
-  )
   (wire (pts (xy 110.49 80.01) (xy 138.43 80.01))
     (stroke (width 0) (type default))
@@
   )
   (wire (pts (xy 105.41 118.11) (xy 105.41 120.65))
+    (stroke (width 0) (type default))
+  )
+  (wire (pts (xy 60.96 130.81) (xy 93.98 130.81))
     (stroke (width 0) (type default))
   )
@@
     (effects (font (size 1.27 1.27)) (justify right))
   )
-  (symbol (lib_id "power:GND") (at 67.31 144.78 0) (unit 1)
-    (in_bom yes) (on_board yes) (dnp no) (fields_autoplaced)
-    (property "Reference" "#PWR015" (at 67.31 151.13 0)
-      (effects (font (size 1.27 1.27)) hide)
-    )
-    (property "Value" "GND" (at 67.31 149.86 0)
-      (effects (font (size 1.27 1.27)) hide)
-    )
-    (property "Footprint" "" (at 67.31 144.78 0)
-      (effects (font (size 1.27 1.27)) hide)
-    )
-    (property "Datasheet" "" (at 67.31 144.78 0)
-      (effects (font (size 1.27 1.27)) hide)
-    )
-    (pin "1")
-    (instances
-      (project "minimouse"
-        (path "/d8fa4cba-2469-4231-847f-065b6b829f44/0999fad3-9a14-4ede-b729-a71c3dbbdf8e"
-          (reference "#PWR015") (unit 1)
-        )
-      )
-    )
-  )
   (symbol (lib_id "Device:R") (at 168.91 100.33 0) (unit 1)
     (in_bom yes) (on_board yes) (dnp no) (fields_autoplaced)
@@
       (effects (font (size 1.27 1.27)) (justify left))
     )
-    (property "Footprint" "" (at 167.132 100.33 90)
+    (property "Footprint" "Resistor_SMD:R_2512_6332Metric" (at 167.132 100.33 90)
       (effects (font (size 1.27 1.27)) hide)
     )
@@
       (effects (font (size 1.27 1.27)) (justify right))
     )
-    (property "Value" "18K" (at 132.08 127 0)
-      (effects (font (size 1.27 1.27)) (justify right))
-    )
-    (property "Footprint" "" (at 131.318 125.73 90)
+    (property "Value" "47K" (at 132.08 127 0)
+      (effects (font (size 1.27 1.27)) (justify right))
+    )
+    (property "Footprint" "Resistor_SMD:R_0603_1608Metric" (at 131.318 125.73 90)
       (effects (font (size 1.27 1.27)) hide)
     )
@@
       (effects (font (size 1.27 1.27)) (justify right))
     )
-    (property "Value" "1.8K" (at 107.95 125.73 0)
-      (effects (font (size 1.27 1.27)) (justify right))
-    )
-    (property "Footprint" "" (at 107.188 124.46 90)
+    (property "Value" "10K" (at 107.95 125.73 0)
+      (effects (font (size 1.27 1.27)) (justify right))
+    )
+    (property "Footprint" "Resistor_SMD:R_0603_1608Metric" (at 107.188 124.46 90)
       (effects (font (size 1.27 1.27)) hide)
     )
@@
       (effects (font (size 1.27 1.27)))
     )
-    (property "Value" "18K" (at 60.96 88.9 90)
+    (property "Value" "10K" (at 60.96 88.9 90)
       (effects (font (size 1.27 1.27)))
     )
-    (property "Footprint" "" (at 60.96 94.488 90)
+    (property "Footprint" "Resistor_SMD:R_0603_1608Metric" (at 60.96 94.488 90)
       (effects (font (size 1.27 1.27)) hide)
     )
@@
       (effects (font (size 1.27 1.27)) (justify left))
     )
-    (property "Value" "10n" (at 69.85 100.33 0)
-      (effects (font (size 1.27 1.27)) (justify left))
-    )
-    (property "Footprint" "" (at 67.0052 102.87 0)
+    (property "Value" "1n" (at 69.85 100.33 0)
+      (effects (font (size 1.27 1.27)) (justify left))
+    )
+    (property "Footprint" "Capacitor_SMD:C_0603_1608Metric" (at 67.0052 102.87 0)
       (effects (font (size 1.27 1.27)) hide)
     )
@@
       (effects (font (size 1.27 1.27)) (justify right))
     )
-    (property "Value" "18K" (at 107.95 113.03 0)
-      (effects (font (size 1.27 1.27)) (justify right))
-    )
-    (property "Footprint" "" (at 107.188 111.76 90)
+    (property "Value" "10K" (at 107.95 113.03 0)
+      (effects (font (size 1.27 1.27)) (justify right))
+    )
+    (property "Footprint" "Resistor_SMD:R_0603_1608Metric" (at 107.188 111.76 90)
       (effects (font (size 1.27 1.27)) hide)
     )
@@
       (effects (font (size 1.27 1.27)))
     )
-    (property "Value" "2.2m" (at 184.15 53.34 90)
+    (property "Value" "2.2u" (at 184.15 53.34 90)
       (effects (font (size 1.27 1.27)))
     )
-    (property "Footprint" "" (at 187.96 57.4548 0)
+    (property "Footprint" "Capacitor_SMD:C_0603_1608Metric" (at 187.96 57.4548 0)
       (effects (font (size 1.27 1.27)) hide)
     )
@@
       (effects (font (size 1.27 1.27)) (justify left))
     )
-    (property "Footprint" "" (at 225.552 86.36 90)
+    (property "Footprint" "Resistor_SMD:R_2512_6332Metric" (at 225.552 86.36 90)
       (effects (font (size 1.27 1.27)) hide)
     )
@@
       (effects (font (size 1.27 1.27)) (justify left))
     )
-    (property "Footprint" "" (at 139.3952 133.35 0)
+    (property "Footprint" "Capacitor_SMD:C_0603_1608Metric" (at 139.3952 133.35 0)
       (effects (font (size 1.27 1.27)) hide)
     )
@@
     )
   )
-  (symbol (lib_id "Device:C") (at 67.31 137.16 0) (unit 1)
-    (in_bom yes) (on_board yes) (dnp no) (fields_autoplaced)
-    (property "Reference" "CEN1" (at 71.12 135.89 0)
-      (effects (font (size 1.27 1.27)) (justify left))
-    )
-    (property "Value" "1n" (at 71.12 138.43 0)
-      (effects (font (size 1.27 1.27)) (justify left))
-    )
-    (property "Footprint" "" (at 68.2752 140.97 0)
-      (effects (font (size 1.27 1.27)) hide)
-    )
-    (property "Datasheet" "~" (at 67.31 137.16 0)
-      (effects (font (size 1.27 1.27)) hide)
-    )
-    (pin "1")
-    (pin "2")
-    (instances
-      (project "minimouse"
-        (path "/d8fa4cba-2469-4231-847f-065b6b829f44/0999fad3-9a14-4ede-b729-a71c3dbbdf8e"
-          (reference "CEN1") (unit 1)
-        )
-      )
-    )
-  )
   (symbol (lib_id "power:+BATT") (at 177.8 58.42 0) (unit 1)
     (in_bom yes) (on_board yes) (dnp no) (fields_autoplaced)
@@
     )
   )
-  (symbol (lib_id "Device:R") (at 67.31 124.46 180) (unit 1)
-    (in_bom yes) (on_board yes) (dnp no) (fields_autoplaced)
-    (property "Reference" "REN1" (at 69.85 123.19 0)
-      (effects (font (size 1.27 1.27)) (justify right))
-    )
-    (property "Value" "18K" (at 69.85 125.73 0)
-      (effects (font (size 1.27 1.27)) (justify right))
-    )
-    (property "Footprint" "" (at 69.088 124.46 90)
-      (effects (font (size 1.27 1.27)) hide)
-    )
-    (property "Datasheet" "~" (at 67.31 124.46 0)
-      (effects (font (size 1.27 1.27)) hide)
-    )
-    (pin "2")
-    (pin "1")
-    (instances
-      (project "minimouse"
-        (path "/d8fa4cba-2469-4231-847f-065b6b829f44/0999fad3-9a14-4ede-b729-a71c3dbbdf8e"
-          (reference "REN1") (unit 1)
-        )
-      )
-    )
-  )
   (symbol (lib_id "power:GND") (at 160.02 116.84 0) (unit 1)
     (in_bom yes) (on_board yes) (dnp no) (fields_autoplaced)
@@
       (effects (font (size 1.27 1.27)) (justify right))
     )
-    (property "Footprint" "" (at 140.208 116.84 90)
+    (property "Footprint" "Resistor_SMD:R_0603_1608Metric" (at 140.208 116.84 90)
       (effects (font (size 1.27 1.27)) hide)
     )
@@
         )
       )
-    )
-  )
-  (symbol (lib_id "power:+3.3V") (at 67.31 120.65 0) (unit 1)
-    (in_bom yes) (on_board yes) (dnp no)
-    (property "Reference" "#PWR08" (at 67.31 124.46 0)
-      (effects (font (size 1.27 1.27)) hide)
-    )
-    (property "Value" "+3.3V" (at 60.96 118.11 0)
-      (effects (font (size 1.27 1.27)))
-    )
-    (property "Footprint" "" (at 67.31 120.65 0)
-      (effects (font (size 1.27 1.27)) hide)
-    )
-    (property "Datasheet" "" (at 67.31 120.65 0)
-      (effects (font (size 1.27 1.27)) hide)
-    )
-    (pin "1")
-    (instances
-      (project "minimouse"
-        (path "/d8fa4cba-2469-4231-847f-065b6b829f44/0999fad3-9a14-4ede-b729-a71c3dbbdf8e"
-          (reference "#PWR08") (unit 1)
-        )
-      )
