File: minimouse.kicad_pcb (KiCad board)
At the start: 2 copper layers, 90 x 85 mm, 22 parts, among them J1 Conn_ARM_JTAG_SWD_10, J5 Conn_01x02, M1 N20_encoder, M2 N20_encoder, U1 STM32F030C8Tx, U4 HC-SR04

Commit message: salim
Parts:
- added C10: 2.2u, Capacitor_SMD:C_0603_1608Metric, F.Cu at (149.2, 131.7)
- added C11: 2.2u, Capacitor_SMD:C_0603_1608Metric, F.Cu at (162.2, 73.5)
- added C12: 2.2u, Capacitor_SMD:C_0603_1608Metric, F.Cu at (122.7, 99.4)
- added C13: 2.2u, Capacitor_SMD:C_0603_1608Metric, F.Cu at (154.7, 89.4)
- added C13: 2.2u, Capacitor_SMD:C_0603_1608Metric, F.Cu at (184.0, 97.7)
- added C7: 2.2u, Capacitor_SMD:C_0603_1608Metric, F.Cu at (154.6, 69.1)
- added C8: 2.2u, Capacitor_SMD:C_0603_1608Metric, F.Cu at (172.9, 99.9)
- added C9: 2.2u, Capacitor_SMD:C_0603_1608Metric, F.Cu at (166.1, 75.1)
- added CEN0: 1n, Capacitor_SMD:C_0603_1608Metric, F.Cu at (160.2, 92.8)
- added Ctoff0: 22n, Capacitor_SMD:C_0603_1608Metric, F.Cu at (160.3, 96.9)
- added D1: LED, LED_SMD:LED_0603_1608Metric, F.Cu at (173.0, 72.4)
- added J2: Conn_01x04, Connector_PinHeader_2.54mm:PinHeader_1x04_P2.54mm_Vertical, F.Cu at (159.5, 70.2)
- added J3: Conn_01x06, Connector_PinHeader_2.54mm:PinHeader_1x06_P2.54mm_Vertical, F.Cu at (170.2, 90.5)
- added J4: Conn_01x06, Connector_PinHeader_2.54mm:PinHeader_1x06_P2.54mm_Vertical, F.Cu at (125.5, 89.9)
- added R10: 330m, Resistor_SMD:R_2512_6332Metric, F.Cu at (155.7, 105.2)
- added R11: 330m, Resistor_SMD:R_2512_6332Metric, F.Cu at (145.0, 104.6)
- added R12: 100, Resistor_SMD:R_0603_1608Metric, F.Cu at (152.5, 74.9)
- added R13: 100, Resistor_SMD:R_0603_1608Metric, F.Cu at (146.8, 75.0)
- added R14: R, Resistor_SMD:R_0603_1608Metric, F.Cu at (173.0, 70.7)
- added R15: 100, Resistor_SMD:R_0603_1608Metric, F.Cu at (151.7, 94.0)
- added R16: 100, Resistor_SMD:R_0603_1608Metric, F.Cu at (140.5, 88.5)
- added R17: 100, Resistor_SMD:R_0603_1608Metric, F.Cu at (150.1, 93.9)
- added R18: 100, Resistor_SMD:R_0603_1608Metric, F.Cu at (140.5, 86.8)
- added REN0: 10K, Resistor_SMD:R_0603_1608Metric, F.Cu at (154.8, 97.0)
- added REN2: 10K, Resistor_SMD:R_0603_1608Metric, F.Cu at (159.1, 102.9)
- added REN3: 47K, Resistor_SMD:R_0603_1608Metric, F.Cu at (164.8, 94.8)
- added REN4: 10K, Resistor_SMD:R_0603_1608Metric, F.Cu at (163.2, 100.6)
- added Rtoff0: 1K, Resistor_SMD:R_0603_1608Metric, F.Cu at (160.3, 94.7)
- added U2: HC-SR04, minimouse:HC-SR04, F.Cu at (150.0, 67.0)
- added U3: STSPIN240, Package_DFN_QFN:VQFN-16-1EP_3x3mm_P0.5mm_EP1.8x1.8mm, F.Cu at (151.6, 101.5)
- U4: value HC-SR04 -> LP5907MFX-3.3; footprint minimouse:HC-SR04 -> Package_TO_SOT_SMD:SOT-23-5
- moved C5 48.0 mm to (167.7, 69.1)
- moved C1 43.4 mm to (184.7, 83.7)
- moved C3 29.1 mm to (170.8, 79.7)
- moved C4 18.3 mm to (145.0, 80.2), turned to 180 degrees
- moved U4 17.5 mm to (167.3, 71.8)
- moved J1 11.1 mm to (174.5, 79.9)
- moved R1 8.59 mm to (149.7, 72.4)
- moved BOOT0 7.77 mm to (149.7, 75.9)
- moved R8 6.82 mm to (154.4, 74.9)
- moved R9 6.47 mm to (145.0, 75.0)
- moved R7 6.25 mm to (155.1, 94.0)
- moved R6 6.19 mm to (153.4, 94.0)
- moved R5 6.01 mm to (148.5, 94.0)
- moved R4 5.93 mm to (146.8, 94.0)
- moved R3 5.83 mm to (145.0, 94.0)
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Connections:
- R8 pad 1: /mcu/UART1_TX -> /external_uart/EXT_UART_RX
- U1 pad 43: /mcu/UART1_RX -> /external_uart/EXT_UART_TX
- U4 pad 1: GND -> +BATT
- U4 pad 2: /mcu/OUT_B9 -> GND
- U4 pad 3: Net-(U4-ECHO) -> +BATT
- U4 pad 4: +3V3 -> unconnected-(U4-NC-Pad4)

Commit message: saveeeeee
Parts:
- moved J5 59.4 mm to (174.3, 80.1)
- moved C10 59.1 mm to (172.6, 77.4)
- moved C13 44.2 mm to (141.5, 85.3)
- moved C1 43.0 mm to (141.8, 80.5)
- moved J1 15.6 mm to (160.2, 86.0), turned to 180 degrees
- moved C12 12.8 mm to (131.6, 90.2)
- moved J4 12.6 mm to (134.2, 80.8)
- moved C3 10.1 mm to (162.6, 85.6), turned to 90 degrees
- moved R2 6.27 mm to (143.4, 94.0), turned to -90 degrees
- moved REN0 4.44 mm to (157.0, 93.2), turned to 90 degrees
- moved R4 2.21 mm to (146.8, 96.2)
- moved R10 2.03 mm to (156.0, 107.2)
- moved D1 1.93 mm to (171.1, 72.4)
- moved R14 1.91 mm to (171.1, 70.8)
- moved R8 1.23 mm to (153.4, 75.6)
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Routing:
- net +BATT: track 0.00 -> 152.7 mm
- net +3.3V: track 0.00 -> 85.9 mm
- net GND: track 0.00 -> 77.1 mm, vias 0 -> 27
- net /motorB/MA: track 0.00 -> 31.2 mm
- net Net-(J3-Pin_3): track 0.00 -> 31.0 mm, vias 0 -> 2
- net /motorA/MA: track 0.00 -> 26.2 mm
- net /motorB/MB: track 0.00 -> 23.7 mm
- net /motorA/MB: track 0.00 -> 21.8 mm
- net /mcu/IN_B2: track 0.00 -> 21.6 mm
- net Net-(J3-Pin_4): track 0.00 -> 20.5 mm, vias 0 -> 2
- net Net-(U3-TOFF): track 0.00 -> 15.1 mm
- net /mcu/~{RESET}: track 0.00 -> 15.0 mm, vias 0 -> 1
- net Net-(U3-REF): track 0.00 -> 10.8 mm
- net /mcu/SWO: track 0.00 -> 10.2 mm
- net /mcu/TIM15_CH1: track 0.00 -> 9.74 mm
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- added copper zone on B.Cu, net GND

Commit message: salimus
Parts:
- added C14: 0.1u, Capacitor_SMD:C_0603_1608Metric, F.Cu at (124.1, 78.9)
- added J5: Conn_01x02, Connector_PinHeader_2.54mm:PinHeader_1x02_P2.54mm_Vertical, F.Cu at (180.4, 80.1)
- added Q1: PMOS, Package_TO_SOT_SMD:SOT-23-3, F.Cu at (180.5, 86.8)
- added R19: 100K, Resistor_SMD:R_0603_1608Metric, F.Cu at (183.6, 80.0)
- added R20: 10K, Resistor_SMD:R_0603_1608Metric, F.Cu at (183.6, 83.4)
- added SW1: SW_Push, Button_Switch_SMD:SW_Push_1P1T_NO_CK_KSC6xxJ, F.Cu at (127.2, 73.8)
- added TP1: TestPoint, TestPoint:TestPoint_Pad_D2.0mm, F.Cu at (170.8, 86.4)
- added TP2: TestPoint, TestPoint:TestPoint_Pad_D2.0mm, F.Cu at (167.2, 86.4)
- added TP3: TestPoint, TestPoint:TestPoint_Pad_D2.0mm, F.Cu at (169.0, 83.6)
- moved C13 0.99 mm to (155.6, 89.6)
- moved R10 0.71 mm to (156.7, 107.1)
- moved C1 0.38 mm to (141.5, 80.4)
- moved C2 0.38 mm to (141.5, 82.1)
- moved C3 0.31 mm to (162.6, 85.3)
Routing:
- net /mcu/~{RESET}: track 15.0 -> 55.8 mm, vias 1 -> 2
- net +3.3V: track 85.9 -> 101.8 mm, vias 0 -> 1
- net Net-(Q1-G): track 0.00 -> 10.7 mm
- net Net-(J5-Pin_2): track 0.00 -> 7.82 mm
- net +BATT: track 152.7 -> 158.4 mm
- net GND: track 77.1 -> 81.3 mm, vias 27 -> 31
- net /motorB/MA: track 31.2 -> 34.5 mm, vias 0 -> 1
- net /motorB/MB: track 23.7 -> 27.0 mm
- net Net-(U3-SENSEB): track 4.04 -> 4.79 mm
- net /motorA/MA: track 26.2 -> 26.3 mm, vias 0 -> 1
